File: PCB/ParentsHob2HoodController.kicad_sch (KiCad schematic)
At the start: 27 parts, among them J1 Programming_Header, J2 FromController, J3 ToRelays, J4 Conn_IR, J5 Conn_ExtraFan, J6 Conn_01x02, J7 Conn_01x06, Q1 AO3400A, SW1 SW_SPST, U1 MCP3208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

Commit message: Created base plate to protect solder joins from metal housing on fan.
Parts:
- removed C2: 100nF/16V, Capacitor_SMD:C_0805_2012Metric, symbol Device:C_Small
- removed U1: MCP3208, Package_SO:SOIC-16_3.9x9.9mm_P1.27mm, symbol Analog_ADC:MCP3208
Connections:
- net SS is gone; now on net CL_4: U3.14 (PB2)
- net CL_3: now also U3.13 (PB1)
- net CL_5: now also U3.12 (PB0)
- net CL_6: now also U3.11 (PD7)
- net CL_8: now also U3.9 (PD5)
- net RL_5: now also U3.27 (PC4); no longer U3.31 (PD1)
- net RL_6: now also U3.28 (PC5); no longer U3.27 (PC4)
- net RL_8: now also U3.25 (PC2); no longer U3.28 (PC5)
- net CL_7: no longer names the net of RN2.3 (R2)
- net CL_7: no longer J2.7 (Pin_7)
- removed net RL_7: J3.7 (Pin_7), RN1.6 (R5), U3.30 (PD0)
- net S_RX: no longer names the net of U3.10 (PD6)
- net S_RX: no longer J7.4 (Pin_4)
- net S_TX renamed TXD
- net TXD: now also U3.31 (PD1); no longer U3.11 (PD7)
- new net RXD: J7.4 (Pin_4), U3.30 (PD0)
- new net SPECIAL_7: J2.7 (Pin_7), J3.7 (Pin_7)
- no-connect marks 16 -> 19
Other:
- moved on the sheet: C6, C7
